File: viper/viper.kicad_pcb (KiCad board)
At the start: 2 copper layers, 128 parts, among them SW1 SW_Push, SW10 SW_Push, SW11 SW_Push, SW12 SW_Push, SW13 SW_Push, SW14 SW_Push, SW14_1 SW_Push, SW15 SW_Push, SW16 SW_Push, SW17 SW_Push, SW18 SW_Push, SW19 SW_Push, SW2 SW_Push, SW20 SW_Push, SW21 SW_Push, SW22 SW_Push, SW23 SW_Push, SW24 SW_Push, SW25 SW_Push, SW26 SW_Push, SW27 SW_Push, SW28 SW_Push, SW28_1 SW_Push, SW29 SW_Push, SW29_1 SW_Push, SW3 SW_Push, SW30 SW_Push, SW31 SW_Push, SW32 SW_Push, SW33 SW_Push, SW34 SW_Push, SW35 SW_Push, SW36 SW_Push, SW37 SW_Push, SW38 SW_Push, SW39 SW_Push, SW4 SW_Push, SW40 SW_Push, SW41 SW_Push, SW41_1 SW_Push, SW42 SW_Push, SW43 SW_Push, SW43_1 SW_Push, SW44 SW_Push, SW45 SW_Push, SW46 SW_Push, SW47 SW_Push, SW48 SW_Push, SW49 SW_Push, SW5 SW_Push, SW50 SW_Push, SW51 SW_Push, SW52 SW_Push, SW53 SW_Push, SW54 SW_Push, SW55 SW_Push, SW55_1 SW_Push, SW56 SW_Push, SW57 SW_Push, SW58 SW_Push, SW59 SW_Push, SW6 SW_Push, SW60 SW_Push, SW61 SW_Push, SW7 SW_Push, SW8 SW_Push, SW9 SW_Push

Commit message: use example diode placement
Parts:
- D1, D10, D11, D12, D13, D14, D15, D16, D17, D18, D19, D2, D20, D21, D22, D23, D24, D25, D26, D27, D28, D29, D3, D30, D31, D32, D33, D34, D35, D36, D37, D38, D39, D4, D40, D41, D42, D43, D44, D45, D46, D47, D48, D49, D5, D50, D51, D52, D53, D54, D55, D56, D57, D58, D59, D6, D60, D61, D7, D8, D9: moved to B.Cu
- moved D61 393.8 mm to (338.5, 118.3), turned to 90 degrees
- moved D56 382.9 mm to (367.0, 99.2), turned to 90 degrees
- moved D60 373.2 mm to (314.6, 118.3), turned to 90 degrees
- moved D55 366.7 mm to (350.4, 99.2), turned to 90 degrees
- moved D54 338.1 mm to (314.6, 99.2), turned to 90 degrees
- moved D14 331.2 mm to (357.5, 42.1), turned to 90 degrees
- moved D53 322.4 mm to (295.6, 99.2), turned to 90 degrees
- moved D28 320.3 mm to (362.3, 61.1), turned to 90 degrees
- moved D59 320.0 mm to (233.7, 118.3), turned to 90 degrees
- moved D13 309.1 mm to (328.9, 42.1), turned to 90 degrees
- moved D52 307.8 mm to (276.5, 99.2), turned to 90 degrees
- moved D41 305.9 mm to (355.1, 80.2), turned to 90 degrees
- moved D27 302.8 mm to (338.5, 61.1), turned to 90 degrees
- moved D12 299.3 mm to (309.9, 42.1), turned to 90 degrees
- moved D26 294.9 mm to (319.4, 61.1), turned to 90 degrees
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Routing:
- net ROW2: track 12.8 -> 290.7 mm
- net ROW3: track 0.00 -> 254.8 mm
- net ROW0: track 6.40 -> 257.2 mm
- net ROW1: track 6.40 -> 233.4 mm
- net ROW4: track 0.00 -> 209.5 mm
- net COL2: track 44.2 -> 85.3 mm
- net COL11: track 60.3 -> 81.3 mm
- net COL3: track 43.1 -> 63.2 mm
- net Net-(D55-A): track 0.00 -> 8.45 mm
- net Net-(D54-A): track 0.00 -> 8.45 mm
- net Net-(D52-A): track 0.00 -> 8.45 mm
- net Net-(D51-A): track 0.00 -> 8.45 mm
- net Net-(D50-A): track 0.00 -> 8.45 mm
- net Net-(D49-A): track 0.00 -> 8.45 mm
- net Net-(D48-A): track 0.00 -> 8.45 mm
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