File: viper_new/viper.kicad_sch (KiCad schematic)
At the start: 274 parts, among them SW1 SW_Push, SW10 SW_Push, SW11 SW_Push, SW12 SW_Push, SW13 SW_Push, SW14 SW_Push, SW14_1 SW_Push, SW15 SW_Push, SW16 SW_Push, SW17 SW_Push, SW18 SW_Push, SW19 SW_Push, SW2 SW_Push, SW20 SW_Push, SW21 SW_Push, SW22 SW_Push, SW23 SW_Push, SW24 SW_Push, SW25 SW_Push, SW26 SW_Push, SW27 SW_Push, SW28 SW_Push, SW28_1 SW_Push, SW29 SW_Push, SW29_1 SW_Push, SW3 SW_Push, SW30 SW_Push, SW31 SW_Push, SW32 SW_Push, SW33 SW_Push, SW34 SW_Push, SW35 SW_Push, SW36 SW_Push, SW37 SW_Push, SW38 SW_Push, SW39 SW_Push, SW4 SW_Push, SW40 SW_Push, SW41 SW_Push, SW41_1 SW_Push, SW42 SW_Push, SW43 SW_Push, SW43_1 SW_Push, SW44 SW_Push, SW45 SW_Push, SW46 SW_Push, SW47 SW_Push, SW48 SW_Push, SW49 SW_Push, SW5 SW_Push, SW50 SW_Push, SW51 SW_Push, SW52 SW_Push, SW53 SW_Push, SW54 SW_Push, SW55 SW_Push, SW55_1 SW_Push, SW56 SW_Push, SW57 SW_Push, SW58 SW_Push, SW59 SW_Push, SW6 SW_Push, SW60 SW_Push, SW61 SW_Push, SW7 SW_Push, SW8 SW_Push, SW9 SW_Push

Commit message: YAKE - YET ANOTHER KEYBOARD EXPORT
Parts:
- added L4: OSH, symbol Mechanical:MountingHole
- D1, D10, D11, D12, D13, D14, D15, D16, D17, D18, D19, D2, D20, D21, D22, D23, D24, D25, D26, D27, D28, D29, D3, D30, D31, D32, D33, D34, D35, D36, D37, D38, D39, D4, D40, D41, D42, D43, D44, D45, D46, D47, D48, D49, D5, D50, D51, D52, D53, D54, D55, D56, D57, D58, D59, D6, D60, D61, D7, D8, D9: footprint Diode_SMD:D_SOD-123 -> Diode_SMD:D_SOD-123F
- H1: value Center Oval Mounting Hole -> Mid Viper Oval Mounting Hole; footprint acheron_MountingHoles:MoutingHole_Oval_7mm_5.0x2.5mm -> acheron_MountingHoles:Mounting_Hole_Oval_2.5x8mm
- H2: value Oval Mounting Hole -> \ Oval Mounting Hole
- H3: value Oval Mounting Hole -> Tab Oval Mounting Hole
- H4: value Mounting Hole -> G-H Mounting Hole; footprint acheron_MountingHoles:MountingHole_2.5x5.0mm -> acheron_MountingHoles:MoutingHole_Oval_BackOnly_7mm_5.0x2.5mm
- H5: value Half Side Hole -> Left Edge Half Side Hole
- H6: value Half Side Hole -> Right Edge Half Side Hole
- H7: value Oval Mounting Hole -> Space Bar Oval Mounting Hole
- H8: value Bottom Half Side Hole -> Left Bottom Half Side Hole
- H9: value Bottom Half Side Hole -> Right Bottom Half Side Hole
- ST14, ST28_1, ST41, ST43, ST55, ST59: now in the parts list
- SW1, SW10, SW11, SW12, SW13, SW14_1, SW16, SW17, SW18, SW19, SW2, SW20, SW21, SW22, SW23, SW24, SW25, SW26, SW27, SW28_1, SW3, SW30, SW31, SW32, SW33, SW34, SW35, SW36, SW37, SW38, SW39, SW4, SW40, SW41_1, SW42, SW44, SW45, SW46, SW47, SW48, SW49, SW5, SW50, SW51, SW52, SW53, SW54, SW56, SW57, SW6, SW61, SW7, SW8, SW9: footprint PCM_Switch_Keyboard_Cherry_MX:SW_Cherry_MX_PCB_1.00u -> PCM_Switch_Keyboard_Hybrid:SW_Hybrid_Cherry_MX_Alps_1.00u
- SW14: footprint PCM_Switch_Keyboard_Cherry_MX:SW_Cherry_MX_PCB_1.00u -> PCM_Switch_Keyboard_Hybrid:SW_Hybrid_Cherry_MX_Alps_2.00u
- SW15, SW28, SW58, SW60: footprint PCM_Switch_Keyboard_Cherry_MX:SW_Cherry_MX_PCB_1.00u -> PCM_Switch_Keyboard_Hybrid:SW_Hybrid_Cherry_MX_Alps_1.50u
- SW29, SW55_1: footprint PCM_Switch_Keyboard_Cherry_MX:SW_Cherry_MX_PCB_1.00u -> PCM_Switch_Keyboard_Hybrid:SW_Hybrid_Cherry_MX_Alps_1.75u
- SW29_1, SW43_1: footprint PCM_Switch_Keyboard_Cherry_MX:SW_Cherry_MX_PCB_1.00u -> PCM_Switch_Keyboard_Hybrid:SW_Hybrid_Cherry_MX_Alps_1.25u
- SW41, SW43: footprint PCM_Switch_Keyboard_Cherry_MX:SW_Cherry_MX_PCB_1.00u -> PCM_Switch_Keyboard_Hybrid:SW_Hybrid_Cherry_MX_Alps_2.25u
- SW55: footprint PCM_Switch_Keyboard_Cherry_MX:SW_Cherry_MX_PCB_1.00u -> PCM_Switch_Keyboard_Hybrid:SW_Hybrid_Cherry_MX_Alps_2.75u
- SW59: footprint PCM_Switch_Keyboard_Cherry_MX:SW_Cherry_MX_PCB_1.00u -> PCM_Switch_Keyboard_Hybrid:SW_Hybrid_Cherry_MX_Alps_7.00u
Other:
- moved on the sheet: LED1, LED10, LED11, LED12, LED13, LED14, LED14_1, LED15, LED16, LED17, LED18, LED19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

Commit message: Added LED matrix & RGB LEDs
Parts:
- added C1, C2: 22p, Capacitor_SMD:C_0603_1608Metric, symbol Device:C_Small
- added C3, C4, C5, C6: 0.1u, Capacitor_SMD:C_0603_1608Metric, symbol Device:C_Small
- added C7: 10u, Capacitor_SMD:C_0603_1608Metric, symbol Device:C_Small
- added C8: 1u, Capacitor_SMD:C_0603_1608Metric, symbol Device:C_Small
- added CRGB1, CRGB2, CRGB3, CRGB4: 100n, Capacitor_SMD:C_0805_2012Metric, symbol Device:C_Small
- added F1: Polyfuse_Small, Fuse:Fuse_1206_3216Metric, symbol Device:Polyfuse_Small
- added J2: USB_B_Mini, acheron_Connectors:USB_MiniB_XM7D-0512, symbol Connector:USB_B_Mini
- added LED62, LED63, LED64, LED65: WS2812B, symbol ws2812b:WS2812B
- added Q1: 2N7002, Package_TO_SOT_SMD:SOT-23, symbol Transistor_FET:2N7002
- added R62, R63: 22, Resistor_SMD:R_0603_1608Metric, symbol Device:R_Small
- added R64, R65: 10k, Resistor_SMD:R_0603_1608Metric, symbol Device:R_Small
- added R66: 1k, Resistor_SMD:R_0603_1608Metric, symbol Device:R_Small
- added RST1: SW_SPST, Button_Switch_SMD:SW_SPST_TL3342, symbol Switch:SW_SPST
- added U1: ATmega32U4-A, Package_QFP:TQFP-44_10x10mm_P0.8mm, symbol MCU_Microchip_ATmega:ATmega32U4-A
- added U2: PRTR5V0U2X, Package_TO_SOT_SMD:SOT-143, symbol Power_Protection:PRTR5V0U2X
- added Y1: Crystal_GND24, Crystal:Crystal_SMD_3225-4Pin_3.2x2.5mm, symbol Device:Crystal_GND24
Connections:
- net +5V: now also C3.1, C4.1, C5.1, C6.1, C7.1, F1.1, R65.2, U1.14 (VCC), U1.2 (UVCC), U1.24 (AVCC), U1.34 (VCC), U1.44 (AVCC), U1.7 (VBUS)
- net COL0: now also U1.20 (PD2)
- net COL1: now also U1.19 (PD1)
- net COL10: now also U1.40 (PF1)
- net COL11: now also U1.39 (PF4)
- net COL12: now also U1.38 (PF5)
- net COL13: now also U1.37 (PF6)
- net COL2: now also U1.18 (PD0)
- net COL3: now also U1.21 (PD3)
- net COL4: now also U1.22 (PD5)
- net COL5: now also U1.29 (PB5)
- net COL6: now also U1.41 (PF0)
- net COL7: now also U1.30 (PB6)
- net COL8: now also U1.31 (PC6)
- net COL9: now also U1.32 (PC7)
- net GND: now also C1.2, C2.2, C3.2, C4.2, C5.2, C6.2, C7.2, C8.2, CRGB1.2, CRGB2.2, CRGB3.2, CRGB4.2, J2.5 (GND), J2.6 (Shield), LED62.3 (GND), LED63.3 (GND), LED64.3 (GND), LED65.3 (GND), Q1.2 (S), R64.2, RST1.1 (A), U1.15 (GND), U1.23 (GND), U1.35 (GND), U1.43 (GND), U1.5 (UGND), U2.1 (GND), Y1.2, Y1.4; no longer LED1.2 (A), LED10.2 (A), LED11.2 (A), LED12.2 (A), LED13.2 (A), LED14.2 (A), LED14_1.2 (A), LED15.2 (A), LED16.2 (A), LED17.2 (A), LED18.2 (A), LED19.2 (A), LED2.2 (A), LED20.2 (A), LED21.2 (A), LED22.2 (A), LED23.2 (A), LED24.2 (A), LED25.2 (A), LED26.2 (A), LED27.2 (A), LED28.2 (A), LED28_1.2 (A), LED29.2 (A), LED29_1.2 (A), LED3.2 (A), LED30.2 (A), LED31.2 (A), LED32.2 (A), LED33.2 (A), LED34.2 (A), LED35.2 (A), LED36.2 (A), LED37.2 (A), LED38.2 (A), LED39.2 (A), LED4.2 (A), LED40.2 (A), LED41.2 (A), LED41_1.2 (A), LED42.2 (A), LED43.2 (A), LED43_1.2 (A), LED44.2 (A), LED45.2 (A), LED46.2 (A), LED47.2 (A), LED48.2 (A), LED49.2 (A), LED5.2 (A), LED50.2 (A), LED51.2 (A), LED52.2 (A), LED53.2 (A), LED54.2 (A), LED55.2 (A), LED55_1.2 (A), LED56.2 (A), LED57.2 (A), LED58.2 (A), LED59.2 (A), LED6.2 (A), LED60.2 (A), LED61.2 (A), LED7.2 (A), LED8.2 (A), LED9.2 (A)
- net ROW0: now also U1.28 (PB4)
- net ROW1: now also U1.27 (PD7)
- net ROW2: now also U1.26 (PD6)
- net ROW3: now also U1.25 (PD4)
- net ROW4: now also U1.1 (PE6)
- new net: R64.1, U1.33 (~{HWB}/PE2)
- new net: Q1.1 (G), R66.1
- new net: R66.2, U1.12 (PB7)
- new net: C8.1, U1.6 (UCAP)
- new net: LED63.2 (DOUT), LED64.4 (DIN)
- new net: LED62.2 (DOUT), LED63.4 (DIN)
- new net: LED64.2 (DOUT), LED65.4 (DIN)
- new net CAPS_LED: U1.8 (PB0)
- new net D+: J2.3 (D+), R62.1, U2.2 (I/O1)
- new net D-: J2.2 (D-), R63.1, U2.3 (I/O2)
- new net LED_GND: LED1.2 (A), LED10.2 (A), LED11.2 (A), LED12.2 (A), LED13.2 (A), LED14.2 (A), LED14_1.2 (A), LED15.2 (A), LED16.2 (A), LED17.2 (A), LED18.2 (A), LED19.2 (A), LED2.2 (A), LED20.2 (A), LED21.2 (A), LED22.2 (A), LED23.2 (A), LED24.2 (A), LED25.2 (A), LED26.2 (A), LED27.2 (A), LED28.2 (A), LED28_1.2 (A), LED29.2 (A), LED29_1.2 (A), LED3.2 (A), LED30.2 (A), LED31.2 (A), LED32.2 (A), LED33.2 (A), LED34.2 (A), LED35.2 (A), LED36.2 (A), LED37.2 (A), LED38.2 (A), LED39.2 (A), LED4.2 (A), LED40.2 (A), LED41.2 (A), LED41_1.2 (A), LED42.2 (A), LED43.2 (A), LED43_1.2 (A), LED44.2 (A), LED45.2 (A), LED46.2 (A), LED47.2 (A), LED48.2 (A), LED49.2 (A), LED5.2 (A), LED50.2 (A), LED51.2 (A), LED52.2 (A), LED53.2 (A), LED54.2 (A), LED55.2 (A), LED55_1.2 (A), LED56.2 (A), LED57.2 (A), LED58.2 (A), LED59.2 (A), LED6.2 (A), LED60.2 (A), LED61.2 (A), LED7.2 (A), LED8.2 (A), LED9.2 (A), Q1.3 (D)
- new net RGB_LED: LED62.4 (DIN), U1.36 (PF7)
- new net USB+: R62.2, U1.4 (D+)
- new net USB-: R63.2, U1.3 (D-)
- new net VCC: CRGB1.1, CRGB2.1, CRGB3.1, CRGB4.1, F1.2, J2.1 (VBUS), LED62.1 (VCC), LED63.1 (VCC), LED64.1 (VCC), LED65.1 (VCC), U2.4 (VCC)
- new net XTAL1: C1.1, U1.17 (XTAL1), Y1.1
- new net XTAL2: C2.1, U1.16 (XTAL2), Y1.3
- new net ~{RESET}: R65.1, RST1.2 (B), U1.13 (~{RESET})
- no-connect marks 0 -> 6
Other:
- note added: "PB1 = SCK PB2 = MOSI PB3 = MISO"
- note added: "RGB Underglow"
- moved on the sheet: H1, H2, H3, H4, H5, H6, H7, H8, H9, L1, L2, L3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

Commit message: Placed parts with respect to SW1
Parts:
- J1: renamed from J2; footprint acheron_Connectors:USB_MiniB_XM7D-0512 -> acheron_Connectors:USB_MiniB_Hirose_UX60-MB-5S8
- LED1, LED10, LED11, LED12, LED13, LED14, LED14_1, LED15, LED16, LED17, LED18, LED19, LED2, LED20, LED21, LED22, LED23, LED24, LED25, LED26, LED27, LED28, LED28_1, LED29, LED29_1, LED3, LED30, LED31, LED32, LED33, LED34, LED35, LED36, LED37, LED38, LED39, LED4, LED40, LED41, LED41_1, LED42, LED43, LED43_1, LED44, LED45, LED46, LED47, LED48, LED49, LED5, LED50, LED51, LED52, LED53, LED54, LED55, LED55_1, LED56, LED57, LED58, LED59, LED6, LED60, LED61, LED7, LED8, LED9: value LED_Small -> LED
- RGB1: renamed from LED62; footprint (none) -> locallib:LED_SMD3528-4P-WS2812B
- RGB2: renamed from LED63; footprint (none) -> locallib:LED_SMD3528-4P-WS2812B
- RGB3: renamed from LED64; footprint (none) -> locallib:LED_SMD3528-4P-WS2812B
- RGB4: renamed from LED65; footprint (none) -> locallib:LED_SMD3528-4P-WS2812B
Connections:
- net +5V: now also F1.2, J1.1 (VBUS), U2.4 (VCC); no longer C3.1, C4.1, C5.1, C6.1, C7.1, F1.1, R1.1, R10.1, R11.1, R12.1, R13.1, R14.1, R15.1, R16.1, R17.1, R18.1, R19.1, R2.1, R20.1, R21.1, R22.1, R23.1, R24.1, R25.1, R26.1, R27.1, R28.1, R29.1, R3.1, R30.1, R31.1, R32.1, R33.1, R34.1, R35.1, R36.1, R37.1, R38.1, R39.1, R4.1, R40.1, R41.1, R42.1, R43.1, R44.1, R45.1, R46.1, R47.1, R48.1, R49.1, R5.1, R50.1, R51.1, R52.1, R53.1, R54.1, R55.1, R56.1, R57.1, R58.1, R59.1, R6.1, R60.1, R61.1, R65.2, R7.1, R8.1, R9.1, U1.14 (VCC), U1.2 (UVCC), U1.24 (AVCC), U1.34 (VCC), U1.44 (AVCC), U1.7 (VBUS)
- net CAPS_LED: now also LED29.2 (A), LED29_1.2 (A)
- net LED_GND: no longer LED29.2 (A), LED29_1.2 (A)
- net VCC: now also C3.1, C4.1, C5.1, C6.1, C7.1, F1.1, R1.1, R10.1, R11.1, R12.1, R13.1, R14.1, R15.1, R16.1, R17.1, R18.1, R19.1, R2.1, R20.1, R21.1, R22.1, R23.1, R24.1, R25.1, R26.1, R27.1, R28.1, R29.1, R3.1, R30.1, R31.1, R32.1, R33.1, R34.1, R35.1, R36.1, R37.1, R38.1, R39.1, R4.1, R40.1, R41.1, R42.1, R43.1, R44.1, R45.1, R46.1, R47.1, R48.1, R49.1, R5.1, R50.1, R51.1, R52.1, R53.1, R54.1, R55.1, R56.1, R57.1, R58.1, R59.1, R6.1, R60.1, R61.1, R65.2, R7.1, R8.1, R9.1, U1.14 (VCC), U1.2 (UVCC), U1.24 (AVCC), U1.34 (VCC), U1.44 (AVCC), U1.7 (VBUS); no longer F1.2, J1.1 (VBUS), U2.4 (VCC)
- net at Q1.1 (G): now also R66.2; no longer R66.1
- net at U1.12 (PB7): now also R66.1; no longer R66.2
Other:
- note added: "Crystal Circuit"
- note added: "Decoupling Capacitors"
- note added: "ESD Circuit"
- note added: "Hard Reset Circuit"
- note added: "RGB Underglow Circuit"
- note added: "USB Circuit"
- note removed: "RGB Underglow"
- moved on the sheet: C1, C2, C3, C4, C5, C6, C7, CRGB1, CRGB2, CRGB3, CRGB4, F1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

Commit message: and the story continues
Parts:
- D1, D10, D11, D12, D13, D14, D15, D16, D17, D18, D19, D2, D20, D21, D22, D23, D24, D25, D26, D27, D28, D29, D3, D30, D31, D32, D33, D34, D35, D36, D37, D38, D39, D4, D40, D41, D42, D43, D44, D45, D46, D47, D48, D49, D5, D50, D51, D52, D53, D54, D55, D56, D57, D58, D59, D6, D60, D61, D7, D8, D9: value D -> 1n4148
- H1, H2, H3, H4, H5, H6, H7, H8, H9: now not fitted; now left out of the parts list
- J1, L1, L2, L3, L4: now left out of the parts list
- R1, R10, R11, R12, R13, R14, R15, R16, R17, R18, R19, R2, R20, R21, R22, R23, R24, R25, R26, R27, R28, R29, R3, R30, R31, R32, R33, R34, R35, R36, R37, R38, R39, R4, R40, R41, R42, R43, R44, R45, R46, R47, R48, R49, R5, R50, R51, R52, R53, R54, R55, R56, R57, R58, R59, R6, R60, R61, R7, R8, R9: value R_Small -> 470; now not fitted
- ST14: value Backspace Stabilizer -> 2u Backspace Stabilizer
- ST28_1: value ISO Enter Stabilizer -> 2u ISO Enter Stabilizer
- ST41: value Enter Stabilizer -> 2u Enter Stabilizer
- ST43: value Left Shift Stabilizer -> 2u Left Shift Stabilizer
- ST55: value Right Shift Stabilizer -> 2u Right Shift Stabilizer
- ST59: value Space Bar Stabilizer -> 7 Space Bar Stabilizer
- SW1, SW10, SW11, SW12, SW13, SW14, SW14_1, SW15, SW16, SW17, SW18, SW19, SW2, SW20, SW21, SW22, SW23, SW24, SW25, SW26, SW27, SW28, SW28_1, SW29, SW29_1, SW3, SW30, SW31, SW32, SW33, SW34, SW35, SW36, SW37, SW38, SW39, SW4, SW40, SW41, SW41_1, SW42, SW43, SW43_1, SW44, SW45, SW46, SW47, SW48, SW49, SW5, SW50, SW51, SW52, SW53, SW54, SW55, SW55_1, SW56, SW57, SW58, SW59, SW6, SW60, SW61, SW7, SW8, SW9: value SW_Push -> Cherry Alps Hybrid
Other:
- moved on the sheet: C1, C2, C3, C4, C5, C6, C7, C8, CRGB1, CRGB2, CRGB3, CRGB4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
