File: hardware/viper_splithhkb/viper-split-hhkb.kicad_pcb (KiCad board)
At the start: 2 copper layers, 285 x 95.1 mm, 188 parts, among them Q1 2N7002, SW1 5.2x5.2mm, SW1 SW_Push, SW10 SW_Push, SW11 SW_Push, SW12 SW_Push, SW13 SW_Push, SW14 SW_Push, SW14_1 SW_Push, SW15 SW_Push, SW16 SW_Push, SW17 SW_Push, SW18 SW_Push, SW19 SW_Push, SW2 SW_Push, SW20 SW_Push, SW21 SW_Push, SW22 SW_Push, SW23 SW_Push, SW24 SW_Push, SW25 SW_Push, SW26 SW_Push, SW27 SW_Push, SW28 SW_Push, SW29 SW_Push, SW29_1 SW_Push, SW3 SW_Push, SW30 SW_Push, SW31 SW_Push, SW32 SW_Push, SW33 SW_Push, SW34 SW_Push, SW35 SW_Push, SW36 SW_Push, SW37 SW_Push, SW38 SW_Push, SW39 SW_Push, SW4 SW_Push, SW40 SW_Push, SW41 SW_Push, SW42 SW_Push, SW43 SW_Push, SW43_1 SW_Push, SW44 SW_Push, SW45 SW_Push, SW46 SW_Push, SW47 SW_Push, SW48 SW_Push, SW49 SW_Push, SW5 SW_Push, SW50 SW_Push, SW51 SW_Push, SW52 SW_Push, SW53 SW_Push, SW54 SW_Push, SW55 SW_Push, SW55_1 SW_Push, SW56 SW_Push, SW57 SW_Push, SW58 SW_Push, SW59 SW_Push, SW59_1 SW_Push, SW6 SW_Push, SW60 SW_Push, SW61 SW_Push, SW62 SW_Push, SW63 SW_Push, SW7 SW_Push, SW8 SW_Push, SW9 SW_Push, U1 ATmega32U4-MU, U2 PRTR5V0U2X, Y1 16Mhz

Commit message: Manually corrected split-hhkb layout
Parts:
- removed C1, C10, C11, C12, C13, C14, C15, C16, C17, C18, C19, C20, C21, C3, C4, C5, C9: 0.1uF, Capacitors_SMD:C_0603
- removed C2: 10uF, Capacitors_SMD:C_0603
- removed C6: 1uF, Capacitors_SMD:C_0603
- removed C7, C8: 22pF, Capacitors_SMD:C_0603
- removed D63: D, Diode_SMD:D_SOD-123F
- removed F1: 500mA, Fuse_Holders_and_Fuses:Fuse_SMD1206_Reflow
- removed Q1: 2N7002, TO_SOT_Packages_SMD:SOT-23
- removed R67, R68: 22, Resistors_SMD:R_0805
- removed R69, R71: 1k, Resistors_SMD:R_0805
- removed R70: 10k, Resistors_SMD:R_0805
- removed R73, R74: 5.1k, Resistors_SMD:R_0805
- removed REF**: viper_outline, locallib:viper_outline
- removed RGB1, RGB10, RGB11, RGB12, RGB13, RGB14, RGB2, RGB3, RGB4, RGB5, RGB6, RGB7, RGB8, RGB9: WS2812B, WS2812B:WS2812B
- removed ST55: MountingHole, Mounting_Keyboard_Stabilizer:Stabilizer_Cherry_MX_2.00u
- removed ST59_1, ST61: MountingHole, Mounting_Keyboard_Stabilizer:Stabilizer_Cherry_MX_3.00u
- removed the SW1 at (95.2, 38.1)
- removed the SW1 at (134.9, 106.5)
- removed SW43_1: SW_Push, Switch_Keyboard_Hybrid:SW_Hybrid_Cherry_MX_Alps_1.25u
- removed SW55_1: SW_Push, Switch_Keyboard_Hybrid:SW_Hybrid_Cherry_MX_Alps_1.75u
- removed SW59_1: SW_Push, Switch_Keyboard_Hybrid:SW_Hybrid_Cherry_MX_Alps_3.00u
- removed SW63: SW_Push, Switch_Keyboard_Hybrid:SW_Hybrid_Cherry_MX_Alps_1.00u
- removed U1: ATmega32U4-MU, Housings_DFN_QFN:QFN-44-1EP_7x7mm_Pitch0.5mm
- removed U2: PRTR5V0U2X, locallib:SOT143B
- removed USB1: HRO-TYPE-C-31-M-12, Type-C:HRO-TYPE-C-31-M-12-Assembly
- removed Y1: 16Mhz, Crystals:Crystal_SMD_3225-4pin_3.2x2.5mm
- added ST54: MountingHole, PCM_Mounting_Keyboard_Stabilizer:Stabilizer_Cherry_MX_2.00u, F.Cu at (288.1, 95.2)
- added ST58: MountingHole, PCM_Mounting_Keyboard_Stabilizer:Stabilizer_Cherry_MX_3.00u, F.Cu at (133.3, 114.3)
- added ST60: MountingHole, PCM_Mounting_Keyboard_Stabilizer:Stabilizer_Cherry_MX_3.00u, F.Cu at (209.6, 114.3)
- added SW1: SW_Push, PCM_Switch_Keyboard_Hybrid:SW_Hybrid_Cherry_MX_Alps_1.00u, F.Cu at (38.1, 38.1)
- added SW54_1: SW_Push, PCM_Switch_Keyboard_Hybrid:SW_Hybrid_Cherry_MX_Alps_1.75u, F.Cu at (278.6, 95.2)
- D1, D10, D11, D12, D13, D14, D15, D16, D17, D18, D19, D2, D20, D21, D22, D23, D24, D25, D26, D27, D28, D29, D3, D30, D31, D32, D33, D34, D35, D36, D37, D38, D39, D4, D40, D41, D42, D43, D44, D45, D46, D47, D48, D49, D5, D50, D51, D52, D53, D54, D55, D56, D57, D58, D59, D6, D60, D61, D62, D7, D8, D9: footprint Diode_SMD:D_SOD-123F -> Diode_SMD:D_0805_2012Metric_Pad1.15x1.40mm_HandSolder
- ST14, ST41, ST43: footprint Mounting_Keyboard_Stabilizer:Stabilizer_Cherry_MX_2.00u -> PCM_Mounting_Keyboard_Stabilizer:Stabilizer_Cherry_MX_2.00u
- ST59: footprint Mounting_Keyboard_Stabilizer:Stabilizer_Cherry_MX_7.00u -> PCM_Mounting_Keyboard_Stabilizer:Stabilizer_Cherry_MX_7.00u
- SW10, SW11, SW12, SW13, SW14_1, SW16, SW17, SW18, SW19, SW2, SW20, SW21, SW22, SW23, SW24, SW25, SW26, SW27, SW3, SW30, SW31, SW32, SW33, SW34, SW35, SW36, SW37, SW38, SW39, SW4, SW40, SW42, SW44, SW45, SW46, SW47, SW48, SW49, SW5, SW50, SW51, SW52, SW53, SW56, SW6, SW7, SW8, SW9: footprint Switch_Keyboard_Hybrid:SW_Hybrid_Cherry_MX_Alps_1.00u -> PCM_Switch_Keyboard_Hybrid:SW_Hybrid_Cherry_MX_Alps_1.00u
- SW14: footprint Switch_Keyboard_Hybrid:SW_Hybrid_Cherry_MX_Alps_2.00u -> PCM_Switch_Keyboard_Hybrid:SW_Hybrid_Cherry_MX_Alps_2.00u
- SW15, SW28: footprint Switch_Keyboard_Hybrid:SW_Hybrid_Cherry_MX_Alps_1.50u -> PCM_Switch_Keyboard_Hybrid:SW_Hybrid_Cherry_MX_Alps_1.50u
- SW29: footprint Switch_Keyboard_Hybrid:SW_Hybrid_Cherry_MX_Alps_1.75u -> PCM_Switch_Keyboard_Hybrid:SW_Hybrid_Cherry_MX_Alps_1.75u
- SW29_1: footprint Switch_Keyboard_Hybrid:SW_Hybrid_Cherry_MX_Alps_1.25u -> PCM_Switch_Keyboard_Hybrid:SW_Hybrid_Cherry_MX_Alps_1.25u
- SW41, SW43: footprint Switch_Keyboard_Hybrid:SW_Hybrid_Cherry_MX_Alps_2.25u -> PCM_Switch_Keyboard_Hybrid:SW_Hybrid_Cherry_MX_Alps_2.25u
- SW54: footprint Switch_Keyboard_Hybrid:SW_Hybrid_Cherry_MX_Alps_1.00u -> PCM_Switch_Keyboard_Hybrid:SW_Hybrid_Cherry_MX_Alps_2.75u
- SW55: footprint Switch_Keyboard_Hybrid:SW_Hybrid_Cherry_MX_Alps_2.75u -> PCM_Switch_Keyboard_Hybrid:SW_Hybrid_Cherry_MX_Alps_1.00u
- SW57: footprint Switch_Keyboard_Hybrid:SW_Hybrid_Cherry_MX_Alps_1.00u -> PCM_Switch_Keyboard_Hybrid:SW_Hybrid_Cherry_MX_Alps_1.50u
- SW58: footprint Switch_Keyboard_Hybrid:SW_Hybrid_Cherry_MX_Alps_1.50u -> PCM_Switch_Keyboard_Hybrid:SW_Hybrid_Cherry_MX_Alps_3.00u
- SW59: footprint Switch_Keyboard_Hybrid:SW_Hybrid_Cherry_MX_Alps_7.00u -> PCM_Switch_Keyboard_Hybrid:SW_Hybrid_Cherry_MX_Alps_7.00u
- SW60: footprint Switch_Keyboard_Hybrid:SW_Hybrid_Cherry_MX_Alps_1.00u -> PCM_Switch_Keyboard_Hybrid:SW_Hybrid_Cherry_MX_Alps_3.00u
- SW61: footprint Switch_Keyboard_Hybrid:SW_Hybrid_Cherry_MX_Alps_3.00u -> PCM_Switch_Keyboard_Hybrid:SW_Hybrid_Cherry_MX_Alps_1.50u
- SW62: footprint Switch_Keyboard_Hybrid:SW_Hybrid_Cherry_MX_Alps_1.50u -> PCM_Switch_Keyboard_Hybrid:SW_Hybrid_Cherry_MX_Alps_1.00u
- moved D56 295.9 mm to (71.8, 117.3)
- moved SW56 295.9 mm to (66.7, 114.3)
- moved D15 59.9 mm to (47.9, 60.2)
- moved D43 57.2 mm to (55.1, 98.3)
- moved SW29 57.2 mm to (45.2, 76.2)
- moved D29 57.2 mm to (50.3, 79.2)
- moved D41 57.2 mm to (298.0, 79.2)
- moved D40 57.2 mm to (267.0, 79.2)
- moved D33 57.2 mm to (133.7, 79.2)
- moved D13 57.2 mm to (271.8, 41.1)
- moved ST14 57.2 mm to (295.3, 38.1)
- moved SW13 57.2 mm to (266.7, 38.1)
- moved SW14 57.2 mm to (295.3, 38.1)
- moved SW24 57.2 mm to (219.1, 57.1)
- moved SW39 57.2 mm to (242.9, 76.2)
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Connections:
- net N$10 renamed /N$10
- net N$11 renamed /N$11
- net N$12 renamed /N$12
- net N$13 renamed /N$13
- net N$14 renamed /N$14
- net N$15 renamed /N$15
- net N$16 renamed /N$16
- net N$17 renamed /N$17
- net N$18 renamed /N$18
- net N$19 renamed /N$19
- net N$2 renamed /N$2
- net N$20 renamed /N$20
- net N$21 renamed /N$21
- net N$22 renamed /N$22
- net N$23 renamed /N$23
- net N$24 renamed /N$24
- net N$25 renamed /N$25
- net N$26 renamed /N$26
- net N$27 renamed /N$27
- net N$28 renamed /N$28
- net N$29 renamed /N$29
- net N$3 renamed /N$3
- net N$30 renamed /N$30
- net N$31 renamed /N$31
- net N$32 renamed /N$32
- net N$33 renamed /N$33
- net N$34 renamed /N$34
- net N$35 renamed /N$35
- net N$36 renamed /N$36
- net N$37 renamed /N$37
- net N$38 renamed /N$38
- net N$39 renamed /N$39
- net N$4 renamed /N$4
- net N$40 renamed /N$40
- net N$41 renamed /N$41
- net N$42 renamed /N$42
- net N$43 renamed /N$43
- net N$44 renamed /N$44
- net N$45 renamed /N$45
- net N$46 renamed /N$46
- net N$47 renamed /N$47
- net N$48 renamed /N$48
- net N$49 renamed /N$49
- net N$5 renamed /N$5
- net N$50 renamed /N$50
- net N$51 renamed /N$51
- net N$52 renamed /N$52
- net N$53 renamed /N$53
- net N$54 renamed /N$54
- net N$55 renamed /N$55
- net N$56 renamed /N$56
- net N$57 renamed /N$57
- net N$6 renamed /N$6
- net N$60 renamed /N$60
- net N$61 renamed /N$61
- net N$62 renamed /N$62
- net N$7 renamed /N$7
- net N$8 renamed /N$8
- net N$9 renamed /N$9
- D1 pad 2: N$1 -> /N$1
- D56 pad 1: ROW3 -> ROW4
- D58 pad 2: N$58 -> /N$58
- D59 pad 2: N$59 -> /N$58
- SW19 pad 1: COL4 -> COL3
- SW33 pad 1: COL4 -> COL3
- SW44 pad 1: COL1 -> COL2
- SW45 pad 1: COL2 -> COL3
- SW47 pad 1: COL4 -> COL5
- SW48 pad 1: COL5 -> COL6
- SW49 pad 1: COL6 -> COL7
- SW5 pad 1: COL4 -> COL3
- SW50 pad 1: COL7 -> COL8
- SW51 pad 1: COL8 -> COL9
- SW52 pad 1: COL9 -> COL10
- SW53 pad 1: COL10 -> COL11
- SW54 pad 1: COL11 -> COL12
- SW55 pad 1: COL12 -> COL13
- SW56 pad 1: COL13 -> COL1
- SW57 pad 1: COL1 -> COL2
- SW58 pad 1: COL2 -> COL3
- SW58 pad 2: N$58 -> /N$58
- SW59 pad 2: N$59 -> /N$58
- SW60 pad 1: COL4 -> COL5
- SW61 pad 1: COL5 -> COL11
- SW62 pad 1: COL11 -> COL12
Routing:
- net GND: track 864.6 -> 0.00 mm, vias 24 -> 0
- net +5V: track 674.4 -> 0.00 mm, vias 11 -> 0
- net ROW3: track 529.4 -> 0.00 mm, vias 2 -> 0
- net ROW2: track 290.7 -> 0.00 mm
- net ROW0: track 257.2 -> 0.00 mm
- net ROW1: track 257.2 -> 0.00 mm
- net ROW4: track 209.5 -> 0.00 mm
- net COL3: track 172.3 -> 0.00 mm
- net COL4: track 166.6 -> 0.00 mm
- net COL11: track 162.6 -> 0.00 mm
- net COL10: track 126.4 -> 0.00 mm
- net COL9: track 126.4 -> 0.00 mm
- net COL6: track 126.4 -> 0.00 mm
- net COL8: track 126.4 -> 0.00 mm
- net COL5: track 126.4 -> 0.00 mm
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- removed copper zone on B.Cu, net GND
Other:
- board outline removed
- rule pad_to_mask_clearance: 0.2 -> 0
