File: hardware/viper/viper.kicad_sch (KiCad schematic)
At the start: 52 parts, among them J1 TYPE-C-31-M-12, Q1 2N7002, U1 ATmega32U4-M, U2 USBLC6-2SC6, Y1 16MHz

Commit message: Updated BOM
Start with manufacturing files.
Parts:
- removed L1: 60Ω @ 100 MHz, Inductor_SMD:L_1206_3216Metric_Pad1.42x1.75mm_HandSolder, symbol Device:L_Ferrite_Small
- added C8: 100nF, Capacitor_SMD:C_0805_2012Metric, symbol Device:C_Small
- added CSH1, CSH2: 4.7nF, Capacitor_SMD:C_0805_2012Metric, symbol Device:C_Small
- added DSH1: 1N4007, Diode_SMD:D_SOD-123, symbol Device:D
- added RSH1, RSH2: 1M, Resistor_SMD:R_0805_2012Metric, symbol Device:R_Small
- C1, C2: value 22p -> 22pF; LCSC C22399635 -> C1653
- C3, C4: LCSC C36911366 -> C1591
- C5: LCSC C47117445 -> C1591
- C6: value 10u -> 10uF; LCSC C36911366 -> C96446
- C7: value 1u -> 1uF; LCSC C5254818 -> C29936
- CRGB1, CRGB2, CRGB3, CRGB4: LCSC (none) -> C36911366
- D63: LCSC (none) -> C19077504; TODO ${ERC_ERROR TODO} Calulate proper value -> ${ERC_ERROR TODO} Possibly SMF5.0CA?
- F1: LCSC C70158 -> C2153712
- H1: symbol Mechanical:MountingHole -> Mechanical:MountingHole_Pad
- Q1: value 2N7002 -> AO3400A; symbol Transistor_FET:2N7002 -> Transistor_FET:AO3400A; LCSC (none) -> C7603192
- R63, R67: LCSC C17414 -> C25804
- R64: LCSC (none) -> C17513
- R65, R66: LCSC C25295 -> C23345
- RCC1, RCC2: LCSC C27834 -> C23186
- RGB1, RGB2, RGB3, RGB4: footprint LED_SMD:LED_WS2812B_PLCC4_5.0x5.0mm_P3.2mm -> locallib:LED_WS2812B-Mini_PLCC4_3.5x3.5mm; LCSC (none) -> C5349955
- U1: LCSC (none) -> C112161
Connections:
- net D+: now also R65.2, U1.4 (D+); no longer J1.A6 (D+), J1.B6 (D+), U2.3 (I/O2)
- net D-: now also R66.2, U1.3 (D-); no longer J1.A7 (D-), J1.B7 (D-), U2.1 (I/O1)
- net GND: now also C8.1, CSH1.1, CSH2.1, RSH1.2, RSH2.2
- net VBUS: now also C8.2
- net Earth renamed SHIELD
- net SHIELD: now also CSH1.2, RSH1.1
- net u2/mcu/D+ renamed U2/MCU/D+
- net U2/MCU/D+: no longer R65.2, U1.4 (D+)
- net u2/mcu/D- renamed U2/MCU/D-
- net U2/MCU/D-: no longer R66.2, U1.3 (D-)
- new net: CSH2.2, DSH1.1 (K), RSH2.1
- new net CASE: DSH1.2 (A), H1.1
- new net J1/U2/D+: J1.A6 (D+), J1.B6 (D+), U2.3 (I/O2)
- new net J1/U2/D-: J1.A7 (D-), J1.B7 (D-), U2.1 (I/O1)
Other:
- sheet LED-Matrix: file viper-led-matrix.kicad_sch -> viper-leD-matrix.kicad_sch
- note added: "Case ESD"
- note added: "Shield"
- note removed: "EMI (?)"
- title: (none) -> Psyduck Viper
- moved on the sheet: C1, C2, C3, C4, C5, C6, C7, CRGB1, CRGB2, CRGB3, CRGB4, D63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
