File: hardware/viper/viper.kicad_pcb (KiCad board)
At the start: 2 copper layers, 285 x 95.1 mm, 298 parts, among them J1 USB_B_Mini, Q1 2N7002, SW1 SW_Push, SW10 SW_Push, SW11 SW_Push, SW12 SW_Push, SW13 SW_Push, SW14 SW_Push, SW14_1 SW_Push, SW15 SW_Push, SW16 SW_Push, SW17 SW_Push, SW18 SW_Push, SW19 SW_Push, SW2 SW_Push, SW20 SW_Push, SW21 SW_Push, SW22 SW_Push, SW23 SW_Push, SW24 SW_Push, SW25 SW_Push, SW26 SW_Push, SW27 SW_Push, SW28 SW_Push, SW29 SW_Push, SW29_1 SW_Push, SW3 SW_Push, SW30 SW_Push, SW31 SW_Push, SW32 SW_Push, SW33 SW_Push, SW34 SW_Push, SW35 SW_Push, SW36 SW_Push, SW37 SW_Push, SW38 SW_Push, SW39 SW_Push, SW4 SW_Push, SW40 SW_Push, SW41 SW_Push, SW41_1 SW_Push, SW42 SW_Push, SW43 SW_Push, SW43_1 SW_Push, SW44 SW_Push, SW45 SW_Push, SW46 SW_Push, SW47 SW_Push, SW48 SW_Push, SW49 SW_Push, SW5 SW_Push, SW50 SW_Push, SW51 SW_Push, SW52 SW_Push, SW53 SW_Push, SW54 SW_Push, SW55 SW_Push, SW55_1 SW_Push, SW56 SW_Push, SW57 SW_Push, SW58 SW_Push, SW59 SW_Push, SW6 SW_Push, SW60 SW_Push, SW61 SW_Push, SW7 SW_Push, SW8 SW_Push, SW9 SW_Push, U1 ATmega32U4-A, U2 PRTR5V0U2X, Y1 Crystal_GND24

Commit message: Test with voyager60 pinout & kle2netlist
Mock positions for rgb leds & ferrite bead

Unrouted board with kle2netlist & pos2orient

No per-switch leds yet

Append docker build to existing schematic

Update schematic from PCB

Apply pos2orient file

Add led matrix sheet, marked as DNP

Use Switch_Misc/MX-LED-PolarityMarked in layout2ledschematic job

Disable unneeded symbol/footprint libraries

Added mock mxlockled symbol, dnp

MX-Lock-LED based on MX-LED from ai03-2725/MX_V2

Fixed courtyard of W_Hybrid_Cherry_MX_Alps_1.00u

Started flipping switch symbols for better routing
Parts:
- removed C8: 1u, Capacitor_SMD:C_0603_1608Metric
- removed LED28_1, LED29_1, LED41_1, LED43_1, LED55_1: LED, Switch_Misc:MX-LED-PolarityMarked
- removed ST41: Enter Stabilizer, PCM_Mounting_Keyboard_Stabilizer:Stabilizer_Cherry_MX_2.00u
- removed ST55: Right Shift Stabilizer, PCM_Mounting_Keyboard_Stabilizer:Stabilizer_Cherry_MX_2.00u
- removed SW29_1, SW43_1: SW_Push, PCM_Switch_Keyboard_Hybrid:SW_Hybrid_Cherry_MX_Alps_1.25u
- removed SW41_1: SW_Push, PCM_Switch_Keyboard_Hybrid:SW_Hybrid_Cherry_MX_Alps_1.00u
- removed SW55_1: SW_Push, PCM_Switch_Keyboard_Hybrid:SW_Hybrid_Cherry_MX_Alps_1.75u
- added D62: 1N4148, Diode_SMD:D_0805_2012Metric_Pad1.15x1.40mm_HandSolder, B.Cu at (319.4, 117.8)
- added D63: SMF9.0CA, Diode_SMD:D_SOD-123, B.Cu at (80.1, 44.0)
- added LED30_1: LED, Switch_Misc:MX-LED-PolarityMarked, F.Cu at (78.6, 76.2)
- added LED54_1: LED, Switch_Misc:MX-LED-PolarityMarked, F.Cu at (316.7, 95.2)
- added LED62: LED, Switch_Misc:MX-LED-PolarityMarked, F.Cu at (314.3, 114.3)
- added LF1: Board Outline, locallib:viper_outline, F.Cu at (209.6, 76.2)
- added MX1337: MXLockLed, locallib:MX-Lock-LED-PolarityMarked, F.Cu at (83.3, 76.2)
- added R69: 1k, Resistor_SMD:R_0805_2012Metric, B.Cu at (108.3, 46.0)
- added RCC1: 5.1k, Resistor_SMD:R_0603_1608Metric, B.Cu at (91.0, 42.8)
- added RCC2: 5.1k, Resistor_SMD:R_0603_1608Metric, B.Cu at (91.0, 44.8)
- added ST42: 2u Enter Stabilizer, Mounting_Keyboard_Stabilizer:Stabilizer_Cherry_MX_2.00u, F.Cu at (331.0, 76.2)
- added ST54: 2u Right Shift Stabilizer, Mounting_Keyboard_Stabilizer:Stabilizer_Cherry_MX_2.00u, F.Cu at (326.2, 95.2)
- added ST58: 3u Left Split HHKB Stabilizer, Mounting_Keyboard_Stabilizer:Stabilizer_Cherry_MX_3.00u, F.Cu at (171.4, 114.3)
- added ST59_1: 8u Space Bar Stabilizer, PCM_Mounting_Keyboard_Stabilizer:Stabilizer_Cherry_MX_8.00u, F.Cu at (209.6, 114.3)
- added ST60: 3u Left Split HHKB Stabilizer, Mounting_Keyboard_Stabilizer:Stabilizer_Cherry_MX_3.00u, F.Cu at (247.7, 114.3)
- added SW30_1: SW_Push, locallib:SW_Hybrid_Cherry_MX_Alps_1.00u, F.Cu at (78.6, 76.2)
- added SW54_1: SW_Push, locallib:SW_Hybrid_Cherry_MX_Alps_1.00u, F.Cu at (316.7, 95.2)
- added SW62: SW_Push, locallib:SW_Hybrid_Cherry_MX_Alps_1.00u, F.Cu at (314.3, 114.3)
- C3, C4, C5: value 0.1u -> 100nF
- C6: value 0.1u -> 10u
- C7: value 10u -> 1u
- CRGB1, CRGB2, CRGB3, CRGB4: value 100n -> 100nF
- D1, D10, D11, D12, D13, D14, D15, D16, D17, D18, D19, D2, D20, D21, D22, D23, D24, D25, D26, D27, D28, D29, D3, D30, D31, D32, D33, D34, D35, D36, D37, D38, D39, D4, D40, D41, D42, D43, D44, D45, D46, D47, D48, D49, D5, D50, D51, D52, D53, D54, D55, D56, D57, D58, D59, D6, D60, D61, D7, D8, D9: value D -> 1N4148; footprint Diode_SMD:D_SOD-123F -> Diode_SMD:D_0805_2012Metric_Pad1.15x1.40mm_HandSolder
- F1: value Polyfuse_Small -> 1.5A trip PTC
- J1: value USB_B_Mini -> TYPE-C-31-M-12; footprint acheron_Connectors:USB_MiniB_Hirose_UX60-MB-5S8 -> Connector_USB:USB_C_Receptacle_HRO_TYPE-C-31-M-12
- L1: value Board Outline -> 60Ω @ 100 MHz; footprint locallib:viper_outline -> Inductor_SMD:L_1206_3216Metric_Pad1.42x1.75mm_HandSolder; moved to B.Cu
- R1, R10, R11, R12, R13, R14, R15, R16, R17, R18, R19, R2, R20, R21, R22, R23, R24, R25, R26, R27, R28, R29, R3, R30, R31, R32, R33, R34, R35, R36, R37, R38, R39, R4, R40, R41, R42, R43, R44, R45, R46, R47, R48, R49, R5, R50, R51, R52, R53, R54, R55, R56, R57, R58, R59, R6, R60, R61, R7, R8, R9: value R_Small -> 470; footprint Resistor_SMD:R_1206_3216Metric_Pad1.30x1.75mm_HandSolder -> Resistor_SMD:R_0805_2012Metric
- R62: value 22 -> 470; footprint Resistor_SMD:R_0603_1608Metric -> Resistor_SMD:R_0805_2012Metric
- R64: value 10k -> 22
- R66: value 1k -> 10k
- ST14: value Backspace Stabilizer -> 2u Backspace Stabilizer; footprint PCM_Mounting_Keyboard_Stabilizer:Stabilizer_Cherry_MX_2.00u -> Mounting_Keyboard_Stabilizer:Stabilizer_Cherry_MX_2.00u
- ST43: value Left Shift Stabilizer -> 2u Left Shift Stabilizer; footprint PCM_Mounting_Keyboard_Stabilizer:Stabilizer_Cherry_MX_2.00u -> Mounting_Keyboard_Stabilizer:Stabilizer_Cherry_MX_2.00u
- ST59: value Space Bar Stabilizer -> 7u Space Bar Stabilizer; footprint PCM_Mounting_Keyboard_Stabilizer:Stabilizer_Cherry_MX_7.00u -> Mounting_Keyboard_Stabilizer:Stabilizer_Cherry_MX_7.00u
- SW1, SW10, SW11, SW12, SW13, SW14_1, SW16, SW17, SW18, SW19, SW2, SW20, SW21, SW22, SW23, SW24, SW25, SW26, SW27, SW3, SW30, SW31, SW32, SW33, SW34, SW35, SW36, SW37, SW38, SW39, SW4, SW40, SW42, SW44, SW45, SW46, SW47, SW48, SW49, SW5, SW50, SW51, SW52, SW53, SW54, SW56, SW57, SW6, SW61, SW7, SW8, SW9: footprint PCM_Switch_Keyboard_Hybrid:SW_Hybrid_Cherry_MX_Alps_1.00u -> locallib:SW_Hybrid_Cherry_MX_Alps_1.00u
- SW14: footprint PCM_Switch_Keyboard_Hybrid:SW_Hybrid_Cherry_MX_Alps_2.00u -> locallib:SW_Hybrid_Cherry_MX_Alps_1.00u
- SW15, SW28, SW58, SW60: footprint PCM_Switch_Keyboard_Hybrid:SW_Hybrid_Cherry_MX_Alps_1.50u -> locallib:SW_Hybrid_Cherry_MX_Alps_1.00u
- SW29: footprint PCM_Switch_Keyboard_Hybrid:SW_Hybrid_Cherry_MX_Alps_1.75u -> locallib:SW_Hybrid_Cherry_MX_Alps_1.00u
- SW41, SW43: footprint PCM_Switch_Keyboard_Hybrid:SW_Hybrid_Cherry_MX_Alps_2.25u -> locallib:SW_Hybrid_Cherry_MX_Alps_1.00u
- SW55: footprint PCM_Switch_Keyboard_Hybrid:SW_Hybrid_Cherry_MX_Alps_2.75u -> locallib:SW_Hybrid_Cherry_MX_Alps_1.00u
- SW59: footprint PCM_Switch_Keyboard_Hybrid:SW_Hybrid_Cherry_MX_Alps_7.00u -> locallib:SW_Hybrid_Cherry_MX_Alps_1.00u
- U1: footprint Package_QFP:TQFP-44_10x10mm_P0.8mm -> Package_DFN_QFN:QFN-44-1EP_7x7mm_P0.5mm_EP5.2x5.2mm
- U2: value PRTR5V0U2X -> USBLC6-2SC6; footprint Package_TO_SOT_SMD:SOT-143 -> Package_TO_SOT_SMD:SOT-23-6
- Y1: value Crystal_GND24 -> 16MHz
- moved H5 304.1 mm to (67.0, 85.7)
- moved H6 266.0 mm to (352.1, 85.7)
- moved LED56 257.9 mm to (104.8, 114.3)
- moved SW56 257.9 mm to (104.8, 114.3)
- moved R56 253.3 mm to (104.8, 121.9), turned to 180 degrees
- moved D56 252.5 mm to (109.9, 117.8), turned to 90 degrees
- moved D15 249.0 mm to (348.0, 41.6), turned to 90 degrees
- moved R15 248.4 mm to (342.9, 45.7), turned to 180 degrees
- moved LED15 243.6 mm to (342.9, 38.1)
- moved SW15 243.6 mm to (342.9, 38.1)
- moved D29 241.9 mm to (343.2, 60.6), turned to 90 degrees
- moved R29 241.2 mm to (338.1, 64.8), turned to 180 degrees
- moved LED29 236.5 mm to (338.1, 57.1)
- moved SW29 236.5 mm to (338.1, 57.1)
- moved H8 207.6 mm to (115.3, 123.5)
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Connections:
- net /N$1 renamed Net-(D1-A)
- net /N$10 renamed Net-(D10-A)
- net /N$11 renamed Net-(D11-A)
- net /N$12 renamed Net-(D12-A)
- net /N$13 renamed Net-(D13-A)
- net /N$14 renamed Net-(D14-A)
- net /N$15 renamed Net-(D15-A)
- net /N$16 renamed Net-(D16-A)
- net /N$17 renamed Net-(D17-A)
- net /N$18 renamed Net-(D18-A)
- net /N$19 renamed Net-(D19-A)
- net /N$2 renamed Net-(D2-A)
- net /N$20 renamed Net-(D20-A)
- net /N$21 renamed Net-(D21-A)
- net /N$22 renamed Net-(D22-A)
- net /N$23 renamed Net-(D23-A)
- net /N$24 renamed Net-(D24-A)
- net /N$25 renamed Net-(D25-A)
- net /N$26 renamed Net-(D26-A)
- net /N$27 renamed Net-(D27-A)
- net /N$28 renamed Net-(D28-A)
- net /N$29 renamed Net-(D29-A)
- net /N$3 renamed Net-(D3-A)
- net /N$31 renamed Net-(D31-A)
- net /N$32 renamed Net-(D32-A)
- net /N$33 renamed Net-(D33-A)
- net /N$34 renamed Net-(D34-A)
- net /N$35 renamed Net-(D35-A)
- net /N$36 renamed Net-(D36-A)
- net /N$37 renamed Net-(D37-A)
- net /N$38 renamed Net-(D38-A)
- net /N$39 renamed Net-(D39-A)
- net /N$4 renamed Net-(D4-A)
- net /N$40 renamed Net-(D40-A)
- net /N$41 renamed Net-(D41-A)
- net /N$42 renamed Net-(D42-A)
- net /N$43 renamed Net-(D43-A)
- net /N$44 renamed Net-(D44-A)
- net /N$45 renamed Net-(D45-A)
- net /N$46 renamed Net-(D46-A)
- net /N$47 renamed Net-(D47-A)
- net /N$48 renamed Net-(D48-A)
- net /N$49 renamed Net-(D49-A)
- net /N$5 renamed Net-(D5-A)
- net /N$50 renamed Net-(D50-A)
- net /N$51 renamed Net-(D51-A)
- net /N$52 renamed Net-(D52-A)
- net /N$53 renamed Net-(D53-A)
- net /N$54 renamed Net-(D54-A)
- net /N$55 renamed Net-(D55-A)
- net /N$56 renamed Net-(D56-A)
- net /N$57 renamed Net-(D57-A)
- net /N$58 renamed Net-(D58-A)
- net /N$59 renamed Net-(D59-A)
- net /N$6 renamed Net-(D6-A)
- net /N$60 renamed Net-(D60-A)
- net /N$61 renamed Net-(D61-A)
- net /N$7 renamed Net-(D7-A)
- net /N$8 renamed Net-(D8-A)
- net /N$9 renamed Net-(D9-A)
- C1 pad 1: XTAL1 -> XTAL2
- C2 pad 1: XTAL2 -> XTAL1
- C7 pad 1: VCC -> /UCAP
- D15 pad 1: ROW1 -> ROW0
- D29 pad 1: ROW2 -> ROW1
- D30 pad 2: /N$30 -> Net-(D30-A)
- D56 pad 1: ROW3 -> ROW4
- F1 pad 1: VCC -> /VBUS
- F1 pad 2: +5V -> VCC
- LED29 pad 2: CAPS_LED -> LED_GND
- LED30 pad 2: LED_GND -> CAPS_LED
- R62 pad 1: D+ -> VCC
- R62 pad 2: USB+ -> Net-(LED62-K)
- R63 pad 2: USB- -> D+
- R64 pad 1: Net-(U1-~{HWB}/PE2) -> D+
- R64 pad 2: GND -> D-
- R65 pad 1: ~{RESET} -> /PE2
- R65 pad 2: VCC -> GND
- R66 pad 1: Net-(U1-PB7) -> /~{RESET}
- R66 pad 2: Net-(Q1-G) -> VCC
- RST1 pad 2: ~{RESET} -> /~{RESET}
- SW15 pad 1: COL0 -> COL14
- SW16 pad 1: COL1 -> COL0
- SW17 pad 1: COL2 -> COL1
- SW18 pad 1: COL3 -> COL2
- SW19 pad 1: COL4 -> COL3
- SW20 pad 1: COL5 -> COL4
- SW21 pad 1: COL6 -> COL5
- SW22 pad 1: COL7 -> COL6
- SW23 pad 1: COL8 -> COL7
- SW24 pad 1: COL9 -> COL8
- SW25 pad 1: COL10 -> COL9
- SW26 pad 1: COL11 -> COL10
- SW27 pad 1: COL12 -> COL11
- SW28 pad 1: COL13 -> COL12
- SW29 pad 1: COL0 -> COL13
- SW30 pad 1: COL1 -> Net-(D30-A)
- SW30 pad 2: /N$30 -> COL0
- SW31 pad 1: COL2 -> COL1
- SW32 pad 1: COL3 -> COL2
- SW33 pad 1: COL4 -> COL3
- SW34 pad 1: COL5 -> COL4
- SW35 pad 1: COL6 -> COL5
- SW36 pad 1: COL7 -> COL6
- SW37 pad 1: COL8 -> COL7
- SW38 pad 1: COL9 -> COL8
- SW39 pad 1: COL10 -> COL9
- SW40 pad 1: COL11 -> COL10
- SW41 pad 1: COL12 -> COL11
- SW42 pad 1: COL13 -> COL12
- SW43 pad 1: COL0 -> COL1
- SW44 pad 1: COL1 -> COL2
- SW45 pad 1: COL2 -> COL3
- SW46 pad 1: COL3 -> COL4
- SW47 pad 1: COL4 -> COL5
- SW48 pad 1: COL5 -> COL6
- SW49 pad 1: COL6 -> COL7
- SW50 pad 1: COL7 -> COL8
- SW51 pad 1: COL8 -> COL9
- SW52 pad 1: COL9 -> COL10
- SW53 pad 1: COL10 -> COL11
- SW54 pad 1: COL11 -> COL12
- SW55 pad 1: COL12 -> COL13
- SW56 pad 1: COL13 -> COL2
- SW57 pad 1: COL1 -> COL3
- SW58 pad 1: COL2 -> COL5
- SW59 pad 1: COL3 -> COL7
- SW60 pad 1: COL11 -> COL9
- SW61 pad 1: COL12 -> COL11
- U1 pad 1: ROW4 -> unconnected-(U1-PE6-Pad1)
- U1 pad 10: unconnected-(U1-PB2-Pad10) -> ROW1
- U1 pad 11: unconnected-(U1-PB3-Pad11) -> ROW2
- U1 pad 12: Net-(U1-PB7) -> SWITCH_LED
- U1 pad 13: ~{RESET} -> /~{RESET}
- U1 pad 18: COL2 -> unconnected-(U1-PD0-Pad18)
- U1 pad 19: COL1 -> COL14
- U1 pad 20: COL0 -> RGB_LED
- U1 pad 21: COL3 -> COL13
- U1 pad 22: COL4 -> COL12
- U1 pad 25: ROW3 -> COL11
- U1 pad 26: ROW2 -> COL10
- U1 pad 27: ROW1 -> COL9
- U1 pad 28: ROW0 -> COL8
- U1 pad 29: COL5 -> COL7
- U1 pad 3: USB- -> D-
- U1 pad 30: COL7 -> COL6
- U1 pad 31: COL8 -> COL5
- U1 pad 32: COL9 -> COL4
- U1 pad 33: Net-(U1-~{HWB}/PE2) -> /PE2
- U1 pad 36: RGB_LED -> COL1
- U1 pad 37: COL13 -> COL3
- U1 pad 38: COL12 -> COL2
- U1 pad 39: COL11 -> COL0
- U1 pad 4: USB+ -> D+
- U1 pad 40: COL10 -> ROW4
- U1 pad 41: COL6 -> ROW3
- U1 pad 6: Net-(U1-UCAP) -> /UCAP
- U1 pad 9: unconnected-(U1-PB1-Pad9) -> ROW0
- U2 pad 1: GND -> D-
- U2 pad 2: D+ -> GND
- U2 pad 3: D- -> D+
- U2 pad 4: +5V -> D+
Routing:
- net COL2: track 0.00 -> 92.0 mm
- net COL3: track 0.00 -> 90.0 mm
- net COL5: track 0.00 -> 88.0 mm
- net COL9: track 0.00 -> 88.0 mm
- net COL7: track 0.00 -> 88.0 mm
- net COL11: track 0.00 -> 86.1 mm
- net COL10: track 0.00 -> 67.0 mm
- net COL6: track 0.00 -> 67.0 mm
- net COL4: track 0.00 -> 67.0 mm
- net COL8: track 0.00 -> 67.0 mm
- net COL1: track 0.00 -> 66.4 mm
- net COL12: track 0.00 -> 53.5 mm
- net COL0: track 0.00 -> 45.8 mm
- net COL13: track 0.00 -> 9.52 mm
- net Net-(D55-A): track 0.00 -> 8.33 mm
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
Commit message: Reannotated IC/USB resistors
Parts:
- SW1, SW10, SW11, SW12, SW13, SW14, SW14_1, SW15, SW16, SW17, SW18, SW19, SW2, SW20, SW21, SW22, SW23, SW24, SW25, SW26, SW27, SW28, SW29, SW3, SW30, SW30_1, SW31, SW32, SW33, SW34, SW35, SW36, SW37, SW38, SW39, SW4, SW40, SW41, SW42, SW43, SW44, SW45, SW46, SW47, SW48, SW49, SW5, SW50, SW51, SW52, SW53, SW54, SW54_1, SW55, SW56, SW57, SW58, SW59, SW6, SW60, SW61, SW62, SW7, SW8, SW9: footprint locallib:SW_Hybrid_Cherry_MX_Alps_1.00u -> locallib:SW_Hybrid_Cherry_MX_Alps_1.00u_1
- moved D1 10.2 mm to (81.3, 41.6)
- moved R44 9.88 mm to (114.0, 97.8), turned to 0 degrees
- moved R26 7.21 mm to (271.1, 59.6), turned to 0 degrees
- moved R41 7.21 mm to (295.0, 78.7), turned to 0 degrees
- moved R45 7.21 mm to (133.0, 97.8), turned to 0 degrees
- moved R47 7.21 mm to (171.1, 97.8), turned to 0 degrees
- moved R49 7.21 mm to (209.2, 97.8), turned to 0 degrees
- moved R50 7.21 mm to (228.3, 97.8), turned to 0 degrees
- moved R56 7.21 mm to (99.7, 116.8), turned to 0 degrees
- moved R57 7.21 mm to (123.5, 116.8), turned to 0 degrees
- moved R59 7.21 mm to (204.5, 116.8), turned to 0 degrees
- moved R60 7.21 mm to (242.6, 116.8), turned to 0 degrees
- moved R10 7.21 mm to (242.6, 40.6), turned to 0 degrees
- moved R16 7.21 mm to (75.9, 59.6), turned to 0 degrees
- moved R17 7.21 mm to (99.7, 59.6), turned to 0 degrees
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- renumbered R66 to R63, R69 to R64, R63 to R65, R64 to R66, R65 to R67
Routing:
- net COL2: track 92.0 -> 0.00 mm
- net COL3: track 90.0 -> 0.00 mm
- net COL5: track 88.0 -> 0.00 mm
- net COL9: track 88.0 -> 0.00 mm
- net COL7: track 88.0 -> 0.00 mm
- net COL11: track 86.1 -> 0.00 mm
- net COL10: track 67.0 -> 0.00 mm
- net COL6: track 67.0 -> 0.00 mm
- net COL4: track 67.0 -> 0.00 mm
- net COL8: track 67.0 -> 0.00 mm
- net COL1: track 66.4 -> 0.00 mm
- net COL12: track 53.5 -> 0.00 mm
- net COL0: track 45.8 -> 0.00 mm
- net COL13: track 9.52 -> 0.00 mm
- net Net-(D55-A): track 8.33 -> 0.00 mm
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
Commit message: Imported JP60 board rules & settings
Other:
- rule pad_to_mask_clearance: 0 -> 0.2
Changed lines of the file:
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@@
 	)
 	(setup
-		(pad_to_mask_clearance 0)
+		(stackup
+			(layer "F.SilkS"
+				(type "Top Silk Screen")
+			)
+			(layer "F.Paste"
+				(type "Top Solder Paste")
+			)
+			(layer "F.Mask"
+				(type "Top Solder Mask")
+				(thickness 0.01)
+			)
+			(layer "F.Cu"
+				(type "copper")
+				(thickness 0.035)
+			)
+			(layer "dielectric 1"
+				(type "core")
+				(thickness 1.51)
+				(material "FR4")
+				(epsilon_r 4.5)
+				(loss_tangent 0.02)
+			)
+			(layer "B.Cu"
+				(type "copper")
+				(thickness 0.035)
+			)
+			(layer "B.Mask"
+				(type "Bottom Solder Mask")
+				(thickness 0.01)
+			)
+			(layer "B.Paste"
+				(type "Bottom Solder Paste")
+			)
+			(layer "B.SilkS"
+				(type "Bottom Silk Screen")
+			)
+			(copper_finish "None")
+			(dielectric_constraints no)
+		)
+		(pad_to_mask_clearance 0.2)
+		(solder_mask_min_width 0.25)
 		(allow_soldermask_bridges_in_footprints no)
 		(tenting front back)

Commit message: Updated BOM
Start with manufacturing files.
Parts:
- removed L1: 60Ω @ 100 MHz, Inductor_SMD:L_1206_3216Metric_Pad1.42x1.75mm_HandSolder
- removed MX1337: MXLockLed, locallib:MX-Lock-LED-PolarityMarked
- added C8: 100nF, Capacitor_SMD:C_0805_2012Metric, B.Cu at (89.1, 43.9)
- added CSH1: 4.7nF, Capacitor_SMD:C_0805_2012Metric, B.Cu at (163.9, 31.8)
- added CSH2: 4.7nF, Capacitor_SMD:C_0805_2012Metric, B.Cu at (183.7, 31.9)
- added DSH1: 1N4007, Diode_SMD:D_SOD-123, B.Cu at (181.0, 34.9)
- added LED30_2: LockLED, locallib:MX-Lock-LED-PolarityMarked, F.Cu at (83.3, 76.2)
- added RSH1: 1M, Resistor_SMD:R_0805_2012Metric, B.Cu at (158.9, 31.8)
- added RSH2: 1M, Resistor_SMD:R_0805_2012Metric, B.Cu at (178.7, 31.9)
- C1, C2: value 22p -> 22pF
- C6: value 10u -> 10uF
- C7: value 1u -> 1uF
- D1, D10, D11, D12, D13, D14, D15, D16, D17, D18, D19, D2, D20, D21, D22, D23, D24, D25, D26, D27, D28, D29, D3, D30, D31, D32, D33, D34, D35, D36, D37, D38, D39, D4, D40, D41, D42, D43, D44, D45, D46, D47, D48, D49, D5, D50, D51, D52, D53, D54, D55, D56, D57, D58, D59, D6, D60, D61, D62, D7, D8, D9: footprint Diode_SMD:D_0805_2012Metric_Pad1.15x1.40mm_HandSolder -> Diode_SMD:D_0805_2012Metric
- H1: value Mid Viper Oval Mounting Hole -> ~
- H2: value \ Oval Mounting Hole -> ~
- H3: value Tab Oval Mounting Hole -> ~
- H4: value G-H Mounting Hole -> ~
- H5: value Left Edge Half Side Hole -> ~
- H6: value Right Edge Half Side Hole -> ~
- H7: value Space Bar Oval Mounting Hole -> ~
- H8: value Left Bottom Half Side Hole -> ~
- H9: value Right Bottom Half Side Hole -> ~
- LF1: value Board Outline -> ~
- Q1: value 2N7002 -> AO3400A
- RGB1, RGB2, RGB3, RGB4: footprint locallib:LED_SMD3528-4P-WS2812B -> locallib:LED_WS2812B-Mini_PLCC4_3.5x3.5mm
- ST14: value 2u Backspace Stabilizer -> ~
- ST42: value 2u Enter Stabilizer -> ~
- ST43: value 2u Left Shift Stabilizer -> ~
- ST54: value 2u Right Shift Stabilizer -> ~
- ST58, ST60: value 3u Left Split HHKB Stabilizer -> ~
- ST59: value 7u Space Bar Stabilizer -> ~
- ST59_1: value 8u Space Bar Stabilizer -> ~
- SW1, SW10, SW11, SW12, SW13, SW14, SW14_1, SW15, SW16, SW17, SW18, SW19, SW2, SW20, SW21, SW22, SW23, SW24, SW25, SW26, SW27, SW28, SW29, SW3, SW30, SW30_1, SW31, SW32, SW33, SW34, SW35, SW36, SW37, SW38, SW39, SW4, SW40, SW41, SW42, SW43, SW44, SW45, SW46, SW47, SW48, SW49, SW5, SW50, SW51, SW52, SW53, SW54, SW54_1, SW55, SW56, SW57, SW58, SW59, SW6, SW60, SW61, SW62, SW7, SW8, SW9: footprint locallib:SW_Hybrid_Cherry_MX_Alps_1.00u_1 -> locallib:SW_Hybrid_Cherry_MX_Alps_1.00u
- U1: value ATmega32U4-A -> ATmega32U4-M
- moved CRGB4 1.64 mm to (349.1, 80.2)
- moved CRGB2 1.64 mm to (349.1, 53.2)
- moved CRGB1 1.64 mm to (70.0, 53.2)
- moved CRGB3 1.64 mm to (70.0, 80.2)
Connections:
- net /N$85 renamed Net-(J1-CC1)
- net /N$86 renamed Net-(J1-CC2)
- net /PE2 renamed Net-(U1-~{HWB}/PE2)
- net /UCAP renamed Net-(U1-UCAP)
- net /VBUS renamed VBUS
- net RGB_LED renamed /RGB_LED
- net SWITCH_LED renamed Net-(U1-PB7)
- C1 pad 1: XTAL2 -> /XTAL1
- C2 pad 1: XTAL1 -> /XTAL2
- H1 pad 1: (no net) -> /CASE
- J1 pad A6: D+ -> /J1/U2/D+
- J1 pad A7: D- -> /J1/U2/D-
- J1 pad B6: D+ -> /J1/U2/D+
- J1 pad B7: D- -> /J1/U2/D-
- J1 pad S1: Earth -> /SHIELD
- R65 pad 1: D- -> /U2/MCU/D+
- R65 pad 2: D+ -> /D+
- R66 pad 1: D+ -> /U2/MCU/D-
- R66 pad 2: D- -> /D-
- U1 pad 16: XTAL2 -> /XTAL2
- U1 pad 17: XTAL1 -> /XTAL1
- U1 pad 3: D- -> /D-
- U1 pad 4: D+ -> /D+
- U1 pad 45: (no net) -> GND
- U2 pad 1: D- -> /J1/U2/D-
- U2 pad 3: D+ -> /J1/U2/D+
- U2 pad 4: D+ -> /U2/MCU/D+
- U2 pad 6: D- -> /U2/MCU/D-
- Y1 pad 1: XTAL1 -> /XTAL1
- Y1 pad 3: XTAL2 -> /XTAL2

Commit message: Debugging footprints for cleaner DRC
Set soldermask properties & improved ref placement on back silkscreen

Silkscreen ref placement & forked HRO type-c receptacle due to edge cut

Flipping switches
Parts:
- DSH1: value 1N4007 -> SMF9.0CA
- J1: footprint Connector_USB:USB_C_Receptacle_HRO_TYPE-C-31-M-12 -> locallib:USB_C_Receptacle_HRO_TYPE-C-31-M-12
- LED1, LED10, LED11, LED12, LED13, LED14, LED14_1, LED15, LED16, LED17, LED18, LED19, LED2, LED20, LED21, LED22, LED23, LED24, LED25, LED26, LED27, LED28, LED29, LED3, LED30, LED30_1, LED31, LED32, LED33, LED34, LED35, LED36, LED37, LED38, LED39, LED4, LED40, LED41, LED42, LED43, LED44, LED45, LED46, LED47, LED48, LED49, LED5, LED50, LED51, LED52, LED53, LED54, LED54_1, LED55, LED56, LED57, LED58, LED59, LED6, LED60, LED61, LED62, LED7, LED8, LED9: footprint Switch_Misc:MX-LED-PolarityMarked -> locallib:MX-LED
- LED30_2: footprint locallib:MX-Lock-LED-PolarityMarked -> locallib:MX-Lock-LED
- SW1, SW10, SW11, SW12, SW13, SW14, SW14_1, SW15, SW16, SW17, SW18, SW19, SW2, SW20, SW21, SW22, SW23, SW24, SW25, SW26, SW27, SW28, SW29, SW3, SW30, SW30_1, SW31, SW32, SW33, SW34, SW35, SW36, SW37, SW38, SW39, SW4, SW40, SW41, SW42, SW43, SW44, SW45, SW46, SW47, SW48, SW49, SW5, SW50, SW51, SW52, SW53, SW54, SW54_1, SW55, SW56, SW57, SW58, SW59, SW6, SW60, SW61, SW62, SW7, SW8, SW9: footprint locallib:SW_Hybrid_Cherry_MX_Alps_1.00u -> locallib:SW_Hybrid_Cherry_MX_Alps_1.00u_1
- moved CSH1 58.1 mm to (105.8, 33.7), turned to 90 degrees
- moved RSH1 55.3 mm to (103.6, 33.7), turned to -90 degrees
- moved RCC2 21.4 mm to (75.2, 30.4), turned to 180 degrees
- moved RCC1 19.0 mm to (75.2, 32.2), turned to 0 degrees
- moved D15 11.0 mm to (337.8, 45.7), turned to 0 degrees
- moved D16 11.0 mm to (75.9, 64.8), turned to 0 degrees
- moved D14 11.0 mm to (328.3, 45.7), turned to 0 degrees
- moved R17 10.2 mm to (109.9, 60.6)
- moved R31 10.2 mm to (114.6, 79.7)
- moved R2 10.2 mm to (100.3, 41.6)
- moved DSH1 8.41 mm to (188.8, 31.8), turned to 0 degrees
- moved D27 6.53 mm to (295.3, 64.8), turned to 0 degrees
- moved D52 6.53 mm to (271.5, 102.8), turned to 0 degrees
- moved D55 6.53 mm to (342.9, 102.8), turned to 0 degrees
- moved D58 6.53 mm to (171.4, 121.9), turned to 0 degrees
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- renumbered C7 to C3, C8 to C4, C3 to CB1, C4 to CB2, C5 to CB3, C6 to CB4, C1 to CX1, C2 to CX2, D63 to DF1, R65 to RD1, R66 to RD2, R67 to RHWB1, R64 to RPB1, R63 to RRST1
Connections:
- SW1 pad 1: COL0 -> Net-(D1-A)
- SW1 pad 2: Net-(D1-A) -> COL0
- SW17 pad 1: COL1 -> Net-(D17-A)
- SW17 pad 2: Net-(D17-A) -> COL1
- SW2 pad 1: COL1 -> Net-(D2-A)
- SW2 pad 2: Net-(D2-A) -> COL1
- SW3 pad 1: COL2 -> Net-(D3-A)
- SW3 pad 2: Net-(D3-A) -> COL2
- SW31 pad 1: COL1 -> Net-(D31-A)
- SW31 pad 2: Net-(D31-A) -> COL1
- SW36 pad 1: COL6 -> Net-(D36-A)
- SW36 pad 2: Net-(D36-A) -> COL6
- SW43 pad 1: COL1 -> Net-(D43-A)
- SW43 pad 2: Net-(D43-A) -> COL1
- SW44 pad 1: COL2 -> Net-(D44-A)
- SW44 pad 2: Net-(D44-A) -> COL2
Routing:
- net COL3: track 0.00 -> 90.0 mm
- net COL5: track 0.00 -> 88.0 mm
- net COL9: track 0.00 -> 88.0 mm
- net COL7: track 0.00 -> 88.0 mm
- net COL11: track 0.00 -> 86.1 mm
- net COL10: track 0.00 -> 67.0 mm
- net COL4: track 0.00 -> 67.0 mm
- net COL8: track 0.00 -> 67.0 mm
- net COL1: track 0.00 -> 61.6 mm
- net COL12: track 0.00 -> 53.5 mm
- net COL2: track 0.00 -> 39.1 mm
- net COL6: track 0.00 -> 23.0 mm
- net COL0: track 0.00 -> 20.4 mm
- net Net-(D14-A): track 0.00 -> 13.6 mm
- net COL13: track 0.00 -> 9.52 mm
Other:
- rule pad_to_mask_clearance: 0.2 -> 0.0508
